File: board/dropla-dc/dropla-dc.kicad_pcb (KiCad board)
At the start: 2 copper layers, 42 x 52 mm, 91 parts, among them J11 Conn_01x01, J12 Conn_01x01, J13 Conn_01x01, J14 Conn_01x01, J2 Conn_01x01, J3 Conn_01x01, J4 Conn_01x01, J5 Conn_01x01, J8 Conn_01x01, J9 Conn_01x01, U1 TPP60308-ES1R-S, U2 TPP60308-ES1R-S, U3 TPP60308-ES1R-S, U4 TPP60308-ES1R-S

Commit message: В процесі.
Parts:
- added C30: 10uF, Capacitor_SMD:C_1206_3216Metric, F.Cu at (98.6, 79.0)
- added C31: 10uF, Capacitor_SMD:C_1206_3216Metric, F.Cu at (96.2, 79.0)
- added C34: 10uF, Capacitor_SMD:C_1206_3216Metric, F.Cu at (117.6, 76.2)
- added C35: 10uF, Capacitor_SMD:C_1206_3216Metric, F.Cu at (115.2, 76.2)
- added C38: 22uF, Capacitor_SMD:C_1206_3216Metric, F.Cu at (111.6, 103.8)
- added C39: 22uF, Capacitor_SMD:C_1206_3216Metric, F.Cu at (114.0, 103.8)
- added C42: 22uF, Capacitor_SMD:C_1206_3216Metric, F.Cu at (129.6, 104.6)
- added C43: 22uF, Capacitor_SMD:C_1206_3216Metric, F.Cu at (132.0, 104.6)
- added H1: MountingHole, MountingHole:MountingHole_3.2mm_M3_DIN965, F.Cu at (131.8, 112.8)
- added H2: MountingHole, MountingHole:MountingHole_3.2mm_M3_DIN965, F.Cu at (96.0, 67.0)
- added H3: MountingHole, MountingHole:MountingHole_3.2mm_M3_DIN965, F.Cu at (132.0, 67.0)
- added H4: MountingHole, MountingHole:MountingHole_3.2mm_M3_DIN965, F.Cu at (96.0, 113.0)
- R17: value 294k -> 536k
- R19: value 5.36k -> 53.6k
- R20: value 103k -> 31.6k
- moved J14 4.12 mm to (127.6, 113.0)
- moved J9 3.49 mm to (117.0, 67.4)
- moved L2 3.06 mm to (126.0, 70.0)
- moved J5 2.60 mm to (119.6, 70.8)
- moved R6 2.42 mm to (120.3, 86.2)
- moved C27 2.38 mm to (104.8, 103.4)
- moved J12 2.28 mm to (112.4, 112.0)
- moved C37 2.21 mm to (106.8, 103.8)
- moved C40 2.21 mm to (109.2, 103.8)
- moved R7 2.20 mm to (109.0, 94.6)
- moved D8 2.18 mm to (100.6, 103.2)
- moved R14 2.12 mm to (122.6, 85.6), turned to -90 degrees
- moved C12 1.60 mm to (127.9, 96.6)
- moved R8 1.60 mm to (127.9, 95.0)
- moved J8 1.36 mm to (98.0, 71.3)
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Routing:
- net +12V: track 16.4 -> 22.4 mm
- net +42V: track 21.9 -> 26.7 mm
- net GND: track 9.82 -> 12.7 mm
- net +3.3V: track 12.3 -> 14.7 mm
- net Net-(U2-EN): track 5.92 -> 8.16 mm
- net +5V: track 14.1 -> 15.8 mm
- net Net-(D3-K): track 8.96 -> 10.3 mm
- net Net-(R22-Pad2): track 0.00 -> 1.35 mm
- net Net-(D4-K): track 9.46 -> 10.4 mm
- net Net-(U2-FB): track 4.05 -> 3.34 mm

Commit message: Вважаємо закінчили.
Parts:
- moved C11 1.87 mm to (108.0, 94.4), turned to -90 degrees
- moved C10 1.72 mm to (121.7, 85.6), turned to 90 degrees
- moved C9 1.67 mm to (103.0, 88.3), turned to 90 degrees
- moved J8 1.50 mm to (96.5, 71.4)
- moved C12 1.28 mm to (127.1, 95.6), turned to -90 degrees
- moved R15 0.96 mm to (106.1, 94.2), turned to 90 degrees
- moved R8 0.94 mm to (128.6, 95.6), turned to 90 degrees
- moved R27 0.93 mm to (103.9, 94.2), turned to -90 degrees
- moved R26 0.90 mm to (125.2, 85.6), turned to 90 degrees
- moved R28 0.85 mm to (123.1, 95.0), turned to -90 degrees
- moved R25 0.84 mm to (106.4, 88.3), turned to 90 degrees
- moved R16 0.76 mm to (125.0, 95.1), turned to 90 degrees
- moved D3 0.70 mm to (117.7, 85.6)
- moved R6 0.61 mm to (120.2, 85.6), turned to -90 degrees
- moved R14 0.60 mm to (123.2, 85.6)
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Routing:
- net +12V: track 22.4 -> 12.8 mm
- net GND: track 12.7 -> 7.56 mm, vias 0 -> 16
- net +42V: track 26.7 -> 22.7 mm
- net Net-(U3-EN): track 4.50 -> 6.47 mm
- net Net-(D5-K): track 9.72 -> 11.6 mm
- net Net-(U2-EN): track 8.16 -> 6.28 mm
- net Net-(D4-K): track 10.4 -> 12.2 mm
- net Net-(D3-K): track 10.3 -> 11.9 mm
- net Net-(R22-Pad2): track 1.35 -> 2.41 mm
- net Net-(D2-K): track 9.36 -> 10.1 mm
- net Net-(D1-K): track 40.1 -> 40.8 mm
- net Net-(U4-BOOT): track 8.94 -> 9.59 mm
- net Net-(R21-Pad2): track 1.35 -> 2.00 mm
- net +3.3V: track 14.7 -> 15.3 mm
- net Net-(R24-Pad2): track 1.35 -> 1.89 mm

Commit message: Закінчили.
Parts:
- added FID1: Fiducial, Fiducial:Fiducial_1mm_Mask3mm, F.Cu at (132.6, 70.8)
- added FID2: Fiducial, Fiducial:Fiducial_1mm_Mask3mm, F.Cu at (95.9, 108.8)
- J11: value Conn_01x01 -> V3+
- J12: value Conn_01x01 -> V3-
- J13: value Conn_01x01 -> V4+
- J14: value Conn_01x01 -> V4-
- J2: value Conn_01x01 -> VIN
- J3: value Conn_01x01 -> GND_IN
- J4: value Conn_01x01 -> V1+
- J5: value Conn_01x01 -> V2+
- J8: value Conn_01x01 -> V1-
- J9: value Conn_01x01 -> V2-
- moved J11 0.41 mm to (109.3, 109.0)
- moved J12 0.40 mm to (111.7, 112.0)
- moved C11 0.22 mm to (107.9, 94.2)
- moved R7 0.22 mm to (109.6, 94.2)
- moved C12 0.22 mm to (127.0, 95.4)
- moved J4 0.20 mm to (98.4, 74.8)
- moved R14 0.20 mm to (123.4, 85.6)
- moved R5 0.20 mm to (101.3, 88.3)
- moved R8 0.20 mm to (128.6, 95.4)
- moved J3 0.14 mm to (116.7, 93.3)
- moved C10 0.10 mm to (121.8, 85.6)
- moved C9 0.10 mm to (102.9, 88.3)
- moved R27 0.10 mm to (104.0, 94.2)
- moved R4 0.10 mm to (127.9, 97.9)
Routing:
- net GND: track 7.56 -> 32.4 mm
- net +12V: track 12.8 -> 19.7 mm
- net +3.3V: track 15.3 -> 20.1 mm
- net +5V: track 16.3 -> 20.7 mm
- net +42V: track 22.7 -> 24.8 mm
