File: board/dropla-dc/dropla-dc.kicad_sch (KiCad schematic)
At the start: 91 parts, among them J11 Conn_01x01, J12 Conn_01x01, J13 Conn_01x01, J14 Conn_01x01, J2 Conn_01x01, J3 Conn_01x01, J4 Conn_01x01, J5 Conn_01x01, J8 Conn_01x01, J9 Conn_01x01, U1 TPP60308-ES1R-S, U2 TPP60308-ES1R-S, U3 TPP60308-ES1R-S, U4 TPP60308-ES1R-S

Commit message: В процесі.
Parts:
- added C30, C31, C34, C35: 10uF, Capacitor_SMD:C_1206_3216Metric, symbol Device:C
- added C38, C39, C42, C43: 22uF, Capacitor_SMD:C_1206_3216Metric, symbol Device:C
- added H1, H2, H3, H4: MountingHole, MountingHole:MountingHole_3.2mm_M3_DIN965, symbol Mechanical:MountingHole
- R17: value 294k -> 536k
- R19: value 5.36k -> 53.6k
- R20: value 103k -> 31.6k
Connections:
- net +12V: now also C34.1, C35.1
- net +3.3V: now also C42.1, C43.1
- net +42V: now also C30.1, C31.1
- net +5V: now also C38.1, C39.1
- net GND: now also C30.2, C31.2, C34.2, C35.2, C38.2, C39.2, C42.2, C43.2
Other:
- note added: "Mounting holes"
- moved on the sheet: C1, C10, C11, C12, C13, C14, C15, C16, C17, C18, C19, C2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

Commit message: Закінчили.
Parts:
- added FID1, FID2: Fiducial, Fiducial:Fiducial_1mm_Mask3mm, symbol Mechanical:Fiducial
- J11: value Conn_01x01 -> V3+
- J12: value Conn_01x01 -> V3-
- J13: value Conn_01x01 -> V4+
- J14: value Conn_01x01 -> V4-
- J2: value Conn_01x01 -> VIN
- J3: value Conn_01x01 -> GND_IN
- J4: value Conn_01x01 -> V1+
- J5: value Conn_01x01 -> V2+
- J8: value Conn_01x01 -> V1-
- J9: value Conn_01x01 -> V2-
Other:
- note added: "Fiducials"
Changed lines of the file:
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@@
 		)
 	)
+	(rectangle
+		(start 53.34 167.64)
+		(end 83.82 195.58)
+		(stroke
+			(width 0)
+			(type dot)
+		)
+		(fill
+			(type none)
+		)
+	)
 	(text "Mounting holes"
 		(exclude_from_sim no)
@@
 		)
 	)
+	(text "Fiducials"
+		(exclude_from_sim no)
+		(at 62.23 170.434 0)
+		(effects
+			(font
+				(size 1.27 1.27)
+			)
+		)
+	)
 	(junction
 		(at 54.61 64.77)
@@
 			)
 		)
-		(property "Value" "Conn_01x01"
+		(property "Value" "VIN"
 			(at 34.036 138.43 0)
 			(show_name no)
@@
 			)
 		)
-		(property "Value" "Conn_01x01"
+		(property "Value" "V4+"
 			(at 270.764 138.43 0)
 			(show_name no)
@@
 			)
 		)
-		(property "Value" "Conn_01x01"
+		(property "Value" "V1+"
 			(at 270.764 27.94 0)
 			(show_name no)
@@
 			)
 		)
-		(property "Value" "Conn_01x01"
+		(property "Value" "V2-"
 			(at 272.034 70.866 0)
 			(show_name no)
@@
 			)
 		)
-		(property "Value" "Conn_01x01"
+		(property "Value" "V3+"
 			(at 272.034 101.6 0)
 			(show_name no)
@@
 			)
 		)
-		(property "Value" "Conn_01x01"
+		(property "Value" "V4-"
 			(at 270.764 144.526 0)
 			(show_name no)
@@
 			)
 		)
-		(property "Value" "Conn_01x01"
+		(property "Value" "V3-"
 			(at 272.034 107.696 0)
 			(show_name no)
@@
 			)
 		)
-		(property "Value" "Conn_01x01"
+		(property "Value" "V1-"
 			(at 270.764 34.036 0)
 			(show_name no)
@@
 	)
 	(symbol
+		(lib_id "Mechanical:Fiducial")
+		(at 58.42 184.15 0)
+		(unit 1)
+		(body_style 1)
+		(exclude_from_sim no)
+		(in_bom no)
+		(on_board yes)
+		(in_pos_files yes)
+		(dnp no)
+		(fields_autoplaced yes)
+		(property "Reference" "FID2"
+			(at 60.96 182.8799 0)
+			(show_name no)
+			(do_not_autoplace no)
+			(effects
+				(font
+					(size 1.27 1.27)
+				)
+				(justify left)
+			)
+		)
+		(property "Value" "Fiducial"
+			(at 60.96 185.4199 0)
+			(show_name no)
+			(do_not_autoplace no)
+			(effects
+				(font
+					(size 1.27 1.27)
+				)
+				(justify left)
+			)
+		)
+		(property "Footprint" "Fiducial:Fiducial_1mm_Mask3mm"
+			(at 58.42 184.15 0)
+			(hide yes)
+			(show_name no)
+			(do_not_autoplace no)
+			(effects
+				(font
+					(size 1.27 1.27)
+				)
+			)
+		)
+		(property "Datasheet" ""
+			(at 58.42 184.15 0)
+			(hide yes)
+			(show_name no)
+			(do_not_autoplace no)
+			(effects
+				(font
+					(size 1.27 1.27)
+				)
+			)
+		)
+		(property "Description" "Fiducial Marker"
+			(at 58.42 184.15 0)
+			(hide yes)
+			(show_name no)
+			(do_not_autoplace no)
+			(effects
+				(font
+					(size 1.27 1.27)
+				)
+			)
+		)
+		(instances
+			(project "dropla-dc"
+				(path "/05a11042-efd8-41bf-a962-23b763a44bea"
+					(reference "FID2")
+					(unit 1)
+				)
+			)
+		)
+	)
+	(symbol
 		(lib_id "power:GND")
 		(at 255.27 110.49 0)
@@
 			)
 		)
-		(property "Value" "Conn_01x01"
+		(property "Value" "V2+"
 			(at 272.034 64.77 0)
 			(show_name no)
@@
 	)
 	(symbol
+		(lib_id "Mechanical:Fiducial")
+		(at 58.42 177.8 0)
+		(unit 1)
+		(body_style 1)
+		(exclude_from_sim no)
+		(in_bom no)
+		(on_board yes)
+		(in_pos_files yes)
+		(dnp no)
+		(fields_autoplaced yes)
+		(property "Reference" "FID1"
+			(at 60.96 176.5299 0)
+			(show_name no)
+			(do_not_autoplace no)
+			(effects
+				(font
+					(size 1.27 1.27)
+				)
+				(justify left)
+			)
+		)
+		(property "Value" "Fiducial"
+			(at 60.96 179.0699 0)
+			(show_name no)
+			(do_not_autoplace no)
+			(effects
+				(font
+					(size 1.27 1.27)
+				)
+				(justify left)
+			)
+		)
+		(property "Footprint" "Fiducial:Fiducial_1mm_Mask3mm"
+			(at 58.42 177.8 0)
+			(hide yes)
+			(show_name no)
+			(do_not_autoplace no)
+			(effects
+				(font
+					(size 1.27 1.27)
+				)
+			)
+		)
+		(property "Datasheet" ""
+			(at 58.42 177.8 0)
+			(hide yes)
+			(show_name no)
+			(do_not_autoplace no)
+			(effects
+				(font
+					(size 1.27 1.27)
+				)
+			)
+		)
+		(property "Description" "Fiducial Marker"
+			(at 58.42 177.8 0)
+			(hide yes)
+			(show_name no)
+			(do_not_autoplace no)
+			(effects
+				(font
+					(size 1.27 1.27)
+				)
+			)
+		)
+		(instances
+			(project "dropla-dc"
+				(path "/05a11042-efd8-41bf-a962-23b763a44bea"
+					(reference "FID1")
+					(unit 1)
+				)
+			)
+		)
+	)
+	(symbol
 		(lib_id "power:GND")
 		(at 162.56 121.92 0)
@@
 			)
 		)
-		(property "Value" "Conn_01x01"
+		(property "Value" "GND_IN"
 			(at 34.036 144.526 0)
 			(show_name no)
